File: RocketFlightComputer/main/_autosave-main.kicad_sch (KiCad schematic)
At the start: 70 parts, among them Y1 32.768kHz, Y2 24MHz

Commit message: Preliminary layout done but need to rearrange sd card and such to have the best routing
Parts:
- Y1: footprint footprint:830050789 -> Crystal:Crystal_SMD_2012-2Pin_2.0x1.2mm_HandSoldering
Changed lines of the file:
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@@
 			)
 		)
-		(property "Footprint" "footprint:830050789"
+		(property "Footprint" "Crystal:Crystal_SMD_2012-2Pin_2.0x1.2mm_HandSoldering"
 			(at 212.09 240.03 0)
 			(effects
