File: RocketFlightComputer/main/main.kicad_sch (KiCad schematic)
At the start: 64 parts, among them Q1 DMG2305UX, Y1 32.768kHz, Y2 24MHz

Commit message: Camera and reserve
Parts:
- Resistor1, Resistor2: value 5.1kohms -> 5.1k
Connections:
- net BMP390_SDA1: now also MCU1.J13 (GPIO_AD_B1_11), MCU1.J14 (GPIO_AD_B1_15)
- net at MCU1.C2 (GPIO_EMC_09): no longer R5.2
- net at MCU1.C3 (GPIO_EMC_36): now also R5.2
- net Cam_TX: now reaches MCU1.C5 (GPIO_EMC_31)
- net Reserve_TX2: now reaches MCU1.D13 (GPIO_B1_12)
- net Reserve_RX2: now reaches MCU1.D14 (GPIO_B1_13)
- net Cam_RX: now reaches MCU1.D5 (GPIO_EMC_32)
- net Reserve_TX3: now reaches MCU1.L11 (GPIO_AD_B1_02)
- net Reserve_TX1: now reaches MCU1.L13 (GPIO_AD_B1_10)
- net Reserve_RX3: now reaches MCU1.M12 (GPIO_AD_B1_03)
- net at F1.1: now also USBc1.A4_B9 (VBUS), USBc1.B4_A9 (VBUS)
- no-connect marks 96 -> 88
Other:
- sheet Camera ports: added Cam_RX, Cam_TX; removed none
- sheet Reserved ports: added Reserve_RX1, Reserve_RX2, Reserve_RX3, Reserve_TX1, Reserve_TX2, Reserve_TX3; removed none
- note added: "10"
- note added: "11"
- note added: "12"
- note added: "14"
- note added: "15"
- note added: "20"
- note added: "21"
- note added: "22"
- note added: "23"
- note added: "26"
- note added: "27"
- note added: "28"
- note added: "29"
- note added: "34"
- note added: "35"
- note added: "36"
- note added: "37"
- note added: "38"
- note added: "9"
- note added: "Not necessary since no USB2 external peripheral"
- note removed: "Pas nécéssaire puisque pas de USB2 pour périphériques externes"
- moved on the sheet: C22, D4, F1, R5, USBc1

Commit message: CID documentation and started the PCB editor process
Parts:
- removed D7: IMU LED, LED_SMD:LED_0603_1608Metric_Pad1.05x0.95mm_HandSolder, symbol Device:LED
- added D2: IMU LED, LED_SMD:LED_0603_1608Metric_Pad1.05x0.95mm_HandSolder, symbol Device:LED
Connections:
- net BMP390_SDA1: no longer MCU1.J13 (GPIO_AD_B1_11), MCU1.J14 (GPIO_AD_B1_15)
- net GNDREF: now also D2.1 (K)
- net at MCU1.C3 (GPIO_EMC_36): no longer R5.2
- net at MCU1.E4 (GPIO_EMC_37): no longer R8.2
- net at MCU1.G12 (GPIO_AD_B1_14): now also R8.2
- net at R8.1: now also D2.2 (A)
- new net: MCU1.J14 (GPIO_AD_B1_15), R5.2
- new net Reserve_RX1: MCU1.J13 (GPIO_AD_B1_11)
Other:
- note added: "2"
- note added: "24"
- note added: "3"
- note added: "39"
- note added: "4"
- note added: "40"
- note added: "41"
- moved on the sheet: R34

Commit message: Layout of PCB mostly done
Parts:
- removed F1: 1A, Resistor_SMD:R_0603_1608Metric_Pad0.98x0.95mm_HandSolder, symbol Device:Fuse
- removed Q1: DMG2305UX, footprint:DMG2305UX, symbol DMG2305UX-7:DMG2305UX-7
- removed Resistor1, Resistor2: 5.1k, Resistor_SMD:R_0603_1608Metric_Pad0.98x0.95mm_HandSolder, symbol Device:R
- removed USBc1: USBC_Receptacle_2.0, footprint:GCT_USB4105-GF-A, symbol Connector:USB_C_Receptacle_USB2.0
- added FID1, FID2, FID3, FID4, FID5, FID6, FID7, FID8: Fiducial, Fiducial:Fiducial_1mm_Mask2mm, symbol Mechanical:Fiducial
- added Resistor3, Resistor4: 5.1k, Resistor_SMD:R_0603_1608Metric_Pad0.98x0.95mm_HandSolder, symbol Device:R
- added USB_C_Receptacle_USB2.0_14P1: USBc, Connector_USB:USB_C_Receptacle_GCT_USB4110, symbol Connector:USB_C_Receptacle_USB2.0_14P
- 878-APS6404L-3SQR-SN1: renamed from PSRAM1; value APS6404L-3SQR-SN -> PSRAM
- D1: value LED -> BOOT LED
- KMR241GLFS1: renamed from ResetButton1; value KMR241GLFS -> RESET
- MIMXRT1062DVL6B1: renamed from MCU1; value MIMXRT1062DVL6B -> MCU; footprint footprint:BGA196C65P14X14_1000X1000X152 -> footprint:BGA196C80P14X14_1200X1200X152
- MKL02Z32VFG4: renamed from Bootloader1; value MKL02Z32VFG4 -> BOOT
- TPS62111RSAR1: renamed from 3.3Vregulator1; value TPS62111RSAR -> 3.3Vreg
- W25Q64JVXGIM_TR1: renamed from FlashMemory1; value W25Q64JVXGIM_TR -> FLASH
Connections:
- net 3.3V is gone; now on net +3.3V: MIMXRT1062DVL6B1.N14 (VDDA_ADC_3P3), MIMXRT1062DVL6B1.P12 (VDD_HIGH_IN)
- net +3.3V: now also MIMXRT1062DVL6B1.F10 (NVCC_GPIO_2); no longer C13.1, C8.1, MIMXRT1062DVL6B1.K8 (VDD_USB_CAP)
- net +7.5V: no longer MIMXRT1062DVL6B1.N6 (USB_OTG1_VBUS), MIMXRT1062DVL6B1.P6 (USB_OTG2_VBUS)
- net D+: now also USB_C_Receptacle_USB2.0_14P1.A6 (D+), USB_C_Receptacle_USB2.0_14P1.B6 (D+)
- net D-: now also USB_C_Receptacle_USB2.0_14P1.A7 (D-), USB_C_Receptacle_USB2.0_14P1.B7 (D-)
- net GNDREF: now also MIMXRT1062DVL6B1.N1 (DCDC_GND_1), MIMXRT1062DVL6B1.N2 (DCDC_GND_2), Resistor3.2, Resistor4.2, USB_C_Receptacle_USB2.0_14P1.A1 (GND), USB_C_Receptacle_USB2.0_14P1.A12 (GND), USB_C_Receptacle_USB2.0_14P1.B1 (GND), USB_C_Receptacle_USB2.0_14P1.B12 (GND), USB_C_Receptacle_USB2.0_14P1.S1 (SHIELD)
- net M1M2: now also MIMXRT1062DVL6B1.H9 (VDD_SOC_IN_8)
- net Reserve_CTX: now reaches MIMXRT1062DVL6B1.H13 (GPIO_AD_B1_08)
- net Reserve_CRX: now reaches MIMXRT1062DVL6B1.M13 (GPIO_AD_B1_09)
- net at L1.2: now also MIMXRT1062DVL6B1.N6 (USB_OTG1_VBUS)
- net at L1.1: now also USB_C_Receptacle_USB2.0_14P1.A4 (VBUS), USB_C_Receptacle_USB2.0_14P1.A9 (VBUS), USB_C_Receptacle_USB2.0_14P1.B4 (VBUS), USB_C_Receptacle_USB2.0_14P1.B9 (VBUS)
- new net: Resistor4.1, USB_C_Receptacle_USB2.0_14P1.B5 (CC2)
- new net: Resistor3.1, USB_C_Receptacle_USB2.0_14P1.A5 (CC1)
- new net: C13.1, C8.1, MIMXRT1062DVL6B1.K8 (VDD_USB_CAP)
- no-connect marks 88 -> 81
Other:
- sheet Reserved ports: added Reserve_CRX, Reserve_CTX; removed none
- note added: "Batt(17V to 3.3V) to 3.3V regulator (max 1.5A)"
- note added: "Not necessary (no external usb)"
- note added: "Not necessary (output enable regulator pin EN)"
- note removed: "*Do not connect USB and battery power at the same time"
- note removed: "Batt(17V to 3.3V) or VUSB(5V) to 3.3V regulator (max 1.5A)"

Commit message: Preliminary layout done but need to rearrange sd card and such to have the best routing
Parts:
- Y1, Y2: footprint Crystal:Crystal_SMD_2012-2Pin_2.0x1.2mm -> footprint:830050789
Changed lines of the file:
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@@
 			)
 		)
-		(property "Footprint" "Crystal:Crystal_SMD_2012-2Pin_2.0x1.2mm"
+		(property "Footprint" "footprint:830050789"
 			(at 271.78 294.005 0)
 			(effects
@@
 			)
 		)
-		(property "Footprint" "Crystal:Crystal_SMD_2012-2Pin_2.0x1.2mm"
+		(property "Footprint" "footprint:830050789"
 			(at 212.09 240.03 0)
 			(effects
