File: RocketFlightComputer/main/main.kicad_sch (KiCad schematic)
At the start: 70 parts, among them Y1 32.768kHz, Y2 24MHz

Commit message: Addition of teensy example and milestone on routing completed, missing a few components to connect
Parts:
- L2: footprint Resistor_SMD:R_0603_1608Metric_Pad0.98x0.95mm_HandSolder -> Inductor_SMD:L_1008_2520Metric_Pad1.43x2.20mm_HandSolder
Connections:
- net GNDREF: now also C11.2, C22.1, TPS62111RSAR1.17 (EP); no longer C11.1, C22.2
- net M1M2: now also L4.2; no longer L4.1
- net PyroCH2_3: now also MIMXRT1062DVL6B1.E8 (GPIO_B0_02); no longer MIMXRT1062DVL6B1.G5 (GPIO_EMC_05)
- net PyroCH3_4: now also MIMXRT1062DVL6B1.E7 (GPIO_B0_01); no longer MIMXRT1062DVL6B1.H5 (GPIO_EMC_06)
- net Servo1_PWM: now also MIMXRT1062DVL6B1.C11 (GPIO_B1_02); no longer MIMXRT1062DVL6B1.H3 (GPIO_EMC_08)
- net Servo2_PWM: now also MIMXRT1062DVL6B1.A11 (GPIO_B1_00); no longer MIMXRT1062DVL6B1.D9 (GPIO_B0_10)
- net Servo4_PWM: now also MIMXRT1062DVL6B1.A10 (GPIO_B0_11); no longer MIMXRT1062DVL6B1.A11 (GPIO_B1_00)
- net at MIMXRT1062DVL6B1.G12 (GPIO_AD_B1_14): now also R8.1; no longer R8.2
- net at MIMXRT1062DVL6B1.H4 (GPIO_EMC_07): no longer R3.2
- net at R5.2: now also MIMXRT1062DVL6B1.H3 (GPIO_EMC_08); no longer MIMXRT1062DVL6B1.J14 (GPIO_AD_B1_15)
- net at MIMXRT1062DVL6B1.M1 (DCDC_LP_1), MIMXRT1062DVL6B1.M2 (DCDC_LP_2): now also L4.1; no longer L4.2
- net at MIMXRT1062DVL6B1.M10 (VDD_SNVS_CAP): now also C22.2; no longer C22.1
- net at C10.2: now also C11.1; no longer C11.2
- net at D2.2 (A): now also R8.2; no longer R8.1
- new net: MIMXRT1062DVL6B1.J14 (GPIO_AD_B1_15), R3.2
- no-connect marks 81 -> 80
Other:
- note added: "16"
- note added: "17"
- moved on the sheet: C11, C22, D3, D4, L4, R3, R5, R8

Commit message: First iteration of layout finished, we could call this v0, congratulations! Need an expert to state if layer 4 and layer 3 interations are ok (pwm/ psram/i2c/uart vs power plane 7.5v and 3.3v )
Parts:
- removed D5: GPS LED, LED_SMD:LED_0603_1608Metric_Pad1.05x0.95mm_HandSolder, symbol Device:LED
- removed R6: 470, Resistor_SMD:R_0603_1608Metric_Pad0.98x0.95mm_HandSolder, symbol Device:R
- D3: value 200G ACC LED -> GPS
- D6: value Misc LED -> 200G ACC LED
Connections:
- net Reserve_CRX: no longer names the net of MIMXRT1062DVL6B1.M13 (GPIO_AD_B1_09)
- net Reserve_CTX: no longer names the net of MIMXRT1062DVL6B1.H13 (GPIO_AD_B1_08)
- net Reserve_RX1: no longer names the net of MIMXRT1062DVL6B1.J13 (GPIO_AD_B1_11)
- net Reserve_RX2 renamed Reserve_RX
- net Reserve_RX3: no longer names the net of MIMXRT1062DVL6B1.M12 (GPIO_AD_B1_03)
- net Reserve_TX1: no longer names the net of MIMXRT1062DVL6B1.L13 (GPIO_AD_B1_10)
- net Reserve_TX2 renamed Reserve_TX
- net Reserve_TX3: no longer names the net of MIMXRT1062DVL6B1.L11 (GPIO_AD_B1_02)
- no-connect marks 80 -> 87
Other:
- sheet Reserved ports: added Reserve_RX, Reserve_TX; removed Reserve_CRX, Reserve_CTX, Reserve_RX1, Reserve_RX2, Reserve_RX3, Reserve_TX1, Reserve_TX2, Reserve_TX3

Commit message: First pass of verification and validation of pcb design
Parts:
- R2, R33, R5, R7, R8: value 470 -> 1k
Other:
- note removed: "Check for the LED voltage to current to check resistor value"
- note removed: "Not necessary since no USB2 external peripheral"
Changed lines of the file:
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@@
 		)
 	)
-	(text "VERIFIED"
-		(exclude_from_sim no)
-		(at 469.9 66.04 0)
-		(effects
-			(font
-				(size 1 1)
-				(thickness 0.4)
-				(bold yes)
-			)
-			(justify left bottom)
-		)
-	)
 	(text "0 (RX1)"
 		(exclude_from_sim no)
@@
 	(text "VERIFIED"
 		(exclude_from_sim no)
+		(at 469.138 95.758 0)
+		(effects
+			(font
+				(size 1 1)
+				(thickness 0.4)
+				(bold yes)
+			)
+			(justify left bottom)
+		)
+	)
+	(text "VERIFIED"
+		(exclude_from_sim no)
 		(at 421.64 160.02 0)
 		(effects
@@
 		)
 	)
-	(text "VERIFIED"
-		(exclude_from_sim no)
-		(at 466.725 130.175 0)
-		(effects
-			(font
-				(size 1 1)
-				(thickness 0.4)
-				(bold yes)
-			)
-			(justify left bottom)
-		)
-	)
 	(text "41"
 		(exclude_from_sim no)
@@
 		)
 	)
-	(text "37"
+	(text "VERIFIED"
 		(exclude_from_sim no)
-		(at 281.94 157.48 0)
+		(at 469.138 35.306 0)
 		(effects
 			(font
-				(size 1.27 1.27)
+				(size 1 1)
+				(thickness 0.4)
+				(bold yes)
 			)
 			(justify left bottom)
 		)
 	)
-	(text "29"
+	(text "37"
 		(exclude_from_sim no)
-		(at 283.21 106.68 0)
+		(at 281.94 157.48 0)
 		(effects
 			(font
 				(size 1.27 1.27)
 			)
-			(justify right bottom)
+			(justify left bottom)
 		)
 	)
 	(text "VERIFIED"
 		(exclude_from_sim no)
-		(at 476.25 203.835 0)
+		(at 469.646 66.294 0)
 		(effects
 			(font
@@
 		)
 	)
-	(text "6"
+	(text "29"
 		(exclude_from_sim no)
-		(at 283.21 152.4 0)
+		(at 283.21 106.68 0)
 		(effects
 			(font
 				(size 1.27 1.27)
 			)
-			(justify left bottom)
+			(justify right bottom)
 		)
 	)
 	(text "VERIFIED"
 		(exclude_from_sim no)
-		(at 423.545 95.885 0)
+		(at 423.164 68.072 0)
 		(effects
 			(font
@@
 		)
 	)
+	(text "6"
+		(exclude_from_sim no)
+		(at 283.21 152.4 0)
+		(effects
+			(font
+				(size 1.27 1.27)
+			)
+			(justify left bottom)
+		)
+	)
 	(text "7"
 		(exclude_from_sim no)
@@
 		)
 	)
-	(text "VERIFIED"
-		(exclude_from_sim no)
-		(at 241.3 314.96 0)
-		(effects
-			(font
-				(size 1 1)
-				(thickness 0.4)
-				(bold yes)
-			)
-			(justify left bottom)
-		)
-	)
 	(text "16"
 		(exclude_from_sim no)
@@
 		)
 	)
-	(text "VERIFIED"
-		(exclude_from_sim no)
-		(at 468.63 34.925 0)
-		(effects
-			(font
-				(size 1 1)
-				(thickness 0.4)
-				(bold yes)
-			)
-			(justify left bottom)
-		)
-	)
-	(text "Check for the LED voltage to \ncurrent to check resistor value"
-		(exclude_from_sim no)
-		(at 317.5 180.975 0)
-		(effects
-			(font
-				(size 1.524 1.524)
-				(thickness 0.4)
-				(bold yes)
-			)
-			(justify left bottom)
-		)
-	)
 	(text "34"
 		(exclude_from_sim no)
@@
 		)
 	)
-	(text "VERIFIED"
-		(exclude_from_sim no)
-		(at 13.97 214.63 0)
-		(effects
-			(font
-				(size 1 1)
-				(thickness 0.4)
-				(bold yes)
-			)
-			(justify left bottom)
-		)
-	)
 	(text "33"
 		(exclude_from_sim no)
@@
 		)
 	)
-	(text "VERIFIED"
-		(exclude_from_sim no)
-		(at 469.265 95.25 0)
-		(effects
-			(font
-				(size 1 1)
-				(thickness 0.4)
-				(bold yes)
-			)
-			(justify left bottom)
-		)
-	)
 	(text "38"
 		(exclude_from_sim no)
@@
 		)
 	)
-	(text "VERIFIED"
-		(exclude_from_sim no)
-		(at 419.1 128.905 0)
-		(effects
-			(font
-				(size 1 1)
-				(thickness 0.4)
-				(bold yes)
-			)
-			(justify left bottom)
-		)
-	)
 	(text "5"
 		(exclude_from_sim no)
@@
 		)
 	)
-	(text "VERIFIED"
-		(exclude_from_sim no)
-		(at 422.91 67.31 0)
-		(effects
-			(font
-				(size 1 1)
-				(thickness 0.4)
-				(bold yes)
-			)
-			(justify left bottom)
-		)
-	)
 	(text "2"
 		(exclude_from_sim no)
@@
 		)
 	)
-	(text "Not necessary since no USB2 external peripheral"
-		(exclude_from_sim no)
-		(at 305.435 40.005 0)
-		(effects
-			(font
-				(size 0.762 0.762)
-			)
-			(justify left bottom)
-		)
-	)
 	(text "11"
 		(exclude_from_sim no)
@@
 	(text "VERIFIED"
 		(exclude_from_sim no)
-		(at 132.715 172.72 0)
+		(at 422.402 96.52 0)
 		(effects
 			(font
@@
 		)
 	)
-	(text "VERIFIED"
-		(exclude_from_sim no)
-		(at 120.015 322.58 0)
-		(effects
-			(font
-				(size 1 1)
-				(thickness 0.4)
-				(bold yes)
-			)
-			(justify left bottom)
-		)
-	)
 	(text "Not necessary \n(no external usb)"
 		(exclude_from_sim no)
@@
 			)
 		)
-		(property "Value" "470"
+		(property "Value" "1k"
 			(at 171.704 344.678 90)
 			(effects
@@
 			)
 		)
-		(property "Value" "470"
+		(property "Value" "1k"
 			(at 305.943 265.43 90)
 			(effects
@@
 			)
 		)
-		(property "Value" "470"
+		(property "Value" "1k"
 			(at 244.094 29.21 90)
 			(effects
@@
 			)
 		)
-		(property "Value" "470"
+		(property "Value" "1k"
 			(at 101.6 368.808 90)
 			(effects
@@
 			)
 		)
-		(property "Value" "470"
+		(property "Value" "1k"
 			(at 314.706 148.59 90)
 			(effects

Commit message: Addition of all components in BOM, metal mounting plates, need to check psram if its ok for signals to pass under, all components need a double check
Parts:
- removed L1, L3: 120, Resistor_SMD:R_0603_1608Metric_Pad0.98x0.95mm_HandSolder, symbol Device:FerriteBead
- removed Y2: 24MHz, footprint:830050789, symbol Device:Crystal
- added FB1, FB2: 120, Resistor_SMD:R_0603_1608Metric_Pad0.98x0.95mm_HandSolder, symbol Device:FerriteBead
- added Y5: XRCGB24M000F2P29R0, XRCGB, symbol Crystal:XRCGB24M000F2P29R0
- APS6404L-SQH-SN1: renamed from 878-APS6404L-3SQR-SN1; LCSC (none) -> C7466603
- C1, C28: LCSC (none) -> C70225
- C10: renamed from C11; value 20pF -> 18pF; LCSC (none) -> C1647
- C11: renamed from C12; LCSC (none) -> C70225
- C12: renamed from C13; LCSC (none) -> C106216
- C13: renamed from C14; LCSC (none) -> C106216
- C14: renamed from C15; LCSC (none) -> C19666
- C15: renamed from C16; LCSC (none) -> C19666
- C16: renamed from C17; LCSC (none) -> C19666
- C17: renamed from C18; LCSC (none) -> C106216
- C18: renamed from C19; LCSC (none) -> C106216
- C19: renamed from C6; LCSC (none) -> C106216
- C2: LCSC (none) -> C2762594
- C20, C21, C22, C26, C4, C5: LCSC (none) -> C106216
- C23, C24: value 12pF -> 10pF; LCSC (none) -> C2168929
- C25: LCSC (none) -> C149619
- C27: LCSC (none) -> C19666
- C3: LCSC (none) -> C1592
- C6: renamed from C7; LCSC (none) -> C23630
- C7: renamed from C8; LCSC (none) -> C149619
- C8: renamed from C9; LCSC (none) -> C19666
- C9: renamed from C10; value 20pF -> 18pF; LCSC (none) -> C1647
- D1: renamed from D8; LCSC (none) -> C20433785; Mouser Part Number (none) -> 78-TLMG1100-GS15
- D2: renamed from D1; LCSC (none) -> C20433785; Mouser Part Number (none) -> 78-TLMG1100-GS15
- D3: value GPS -> GPS LED; LCSC (none) -> C20433785; Mouser Part Number (none) -> 78-TLMG1100-GS15
- D4: LCSC (none) -> C20433785; Mouser Part Number (none) -> 78-TLMG1100-GS15
- D5: renamed from D6; LCSC (none) -> C20433785; Mouser Part Number (none) -> 78-TLMG1100-GS15
- D6: renamed from D2; LCSC (none) -> C20433785; Mouser Part Number (none) -> 78-TLMG1100-GS15
- KMR241GLFS1: LCSC (none) -> C221682
- L1: renamed from L2; LCSC (none) -> C307868; Mouser Part Number (none) -> 810-VLS25212HBX6R8M1
- L2: renamed from L4; footprint Resistor_SMD:R_0603_1608Metric_Pad0.98x0.95mm_HandSolder -> Inductor_SMD:L_0805_2012Metric_Pad1.05x1.20mm_HandSolder; LCSC (none) -> C397305; Mouser Part Number (none) -> 81-LQM21PN4R7NGRDRD
- MIMXRT1062DVL6B1: LCSC (none) -> C2847497
- MKL02Z32VFG1: renamed from MKL02Z32VFG4; Mouser Part Number 841-MKL02Z32VFG4 -> (none); now not fitted
- R1: renamed from Resistor3; LCSC (none) -> C1647
- R10: renamed from R4; LCSC (none) -> C18679
- R11: renamed from R8; value 1k -> 470; LCSC (none) -> C23179
- R12: renamed from R7; value 1k -> 470; LCSC (none) -> C23179
- R13: renamed from R9; LCSC (none) -> C14675
- R2: renamed from Resistor4; LCSC (none) -> C1647
- R3: renamed from R1; LCSC (none) -> C22935
- R4: renamed from R33; LCSC (none) -> C21190
- R5: renamed from R2; value 1k -> 470; LCSC (none) -> C23179
- R6: renamed from R34; LCSC (none) -> C23162
- R7: renamed from R3; LCSC (none) -> C23179
- R8: renamed from R11; LCSC (none) -> C23162
- R9: renamed from R5; value 1k -> 470; LCSC (none) -> C23179
- TPS62111RSAR1: LCSC (none) -> C133558
- USB_C_Receptacle_USB2.0_14P1: LCSC (none) -> C5143397; Mouser Part Number (none) -> 640-USB4110-GF-A
- W25Q64JVXGIM_TR1: LCSC (none) -> C7398634
- Y1: LCSC (none) -> C510776; Mouser Part Number (none) -> 815-ABS06-32.7K-9-T
- renumbered FID4 to FID2, FID2 to FID3, FID5 to FID4, FID3 to FID5
Connections:
- net +3.3V: now also FB2.1
- net GNDREF: now also C23.2, Y5.3 (XTAL_2), Y5.4 (NC_2); no longer C23.1
- net N11: now also C23.1, Y5.2 (NC_1); no longer C23.2
- net P11: now also Y5.1 (XTAL_1)
- net at C11.1, C14.1, C18.1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: now also FB2.2
- net at USB_C_Receptacle_USB2.0_14P1.A4 (VBUS), USB_C_Receptacle_USB2.0_14P1.A9 (VBUS), USB_C_Receptacle_USB2.0_14P1.B4 (VBUS)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: now also FB1.1
- net at MIMXRT1062DVL6B1.N6 (USB_OTG1_VBUS): now also FB1.2
Other:
- moved on the sheet: C23, C24, R10

Commit message: Last commit before changing bga to trace clearance of 6mils
Parts:
- FID1, FID2, FID3, FID4, FID5, FID6, FID7, FID8: now not fitted
Other:
- moved on the sheet: R10
Changed lines of the file:
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@@
 	)
 	(junction
+		(at 302.26 346.71)
+		(diameter 0)
+		(color 0 0 0 0)
+	)
+	(junction
 		(at 234.95 186.69)
 		(diameter 0)
@@
 	)
 	(junction
-		(at 302.26 347.98)
-		(diameter 0)
-		(color 0 0 0 0)
-	)
-	(junction
 		(at 229.87 118.11)
 		(diameter 0)
@@
 	(wire
 		(pts
-			(xy 302.26 336.55) (xy 302.26 347.98)
+			(xy 302.26 336.55) (xy 302.26 346.71)
 		)
 		(stroke
@@
 	(wire
 		(pts
+			(xy 302.26 346.71) (xy 302.26 353.06)
+		)
+		(stroke
+			(width 0)
+			(type default)
+		)
+	)
+	(wire
+		(pts
 			(xy 236.22 264.16) (xy 236.22 260.35)
 		)
@@
 	(wire
 		(pts
-			(xy 283.21 336.55) (xy 283.21 347.98)
+			(xy 283.21 336.55) (xy 283.21 346.71)
 		)
 		(stroke
@@
 	(wire
 		(pts
-			(xy 283.21 347.98) (xy 290.83 347.98)
+			(xy 283.21 346.71) (xy 289.56 346.71)
 		)
 		(stroke
@@
 	(wire
 		(pts
-			(xy 302.26 347.98) (xy 298.45 347.98)
+			(xy 302.26 346.71) (xy 297.18 346.71)
 		)
 		(stroke
@@
 	(wire
 		(pts
-			(xy 302.26 347.98) (xy 302.26 353.06)
-		)
-		(stroke
-			(width 0)
-			(type default)
-		)
-	)
-	(wire
-		(pts
 			(xy 317.5 120.65) (xy 303.53 120.65)
 		)
@@
 		(in_bom no)
 		(on_board yes)
-		(dnp no)
+		(dnp yes)
 		(fields_autoplaced yes)
 		(property "Reference" "FID7"
@@
 		(in_bom no)
 		(on_board yes)
-		(dnp no)
+		(dnp yes)
 		(fields_autoplaced yes)
 		(property "Reference" "FID4"
@@
 		(in_bom no)
 		(on_board yes)
-		(dnp no)
+		(dnp yes)
 		(fields_autoplaced yes)
 		(property "Reference" "FID6"
@@
 		(in_bom no)
 		(on_board yes)
-		(dnp no)
+		(dnp yes)
 		(fields_autoplaced yes)
 		(property "Reference" "FID3"
@@
 	(symbol
 		(lib_id "Device:R")
-		(at 294.64 347.98 270)
+		(at 293.37 346.71 270)
 		(unit 1)
 		(exclude_from_sim no)
@@
 		(dnp no)
 		(property "Reference" "R10"
-			(at 288.925 344.17 90)
+			(at 287.655 342.9 90)
 			(effects
 				(font
@@
 		)
 		(property "Value" "2.2M"
-			(at 288.925 346.71 90)
+			(at 287.655 345.44 90)
 			(effects
 				(font
@@
 		)
 		(property "Footprint" "Resistor_SMD:R_0603_1608Metric_Pad0.98x0.95mm_HandSolder"
-			(at 294.64 346.202 90)
+			(at 293.37 344.932 90)
 			(effects
 				(font
@@
 		)
 		(property "Datasheet" "~"
-			(at 294.64 347.98 0)
+			(at 293.37 346.71 0)
 			(effects
 				(font
@@
 		)
 		(property "Description" ""
-			(at 294.64 347.98 0)
+			(at 293.37 346.71 0)
 			(effects
 				(font
@@
 		)
 		(property "LCSC" "C18679 "
-			(at 294.64 347.98 0)
+			(at 293.37 346.71 0)
 			(effects
 				(font
@@
 		(dnp no)
 		(property "Reference" "R11"
-			(at 303.022 264.414 90)
+			(at 311.912 264.414 90)
 			(effects
 				(font
@@
 		)
 		(property "Value" "470"
-			(at 305.943 265.43 90)
+			(at 305.562 265.43 90)
 			(effects
 				(font
@@
 		(in_bom no)
 		(on_board yes)
-		(dnp no)
+		(dnp yes)
 		(fields_autoplaced yes)
 		(property "Reference" "FID8"
@@
 		(in_bom no)
 		(on_board yes)
-		(dnp no)
+		(dnp yes)
 		(fields_autoplaced yes)
 		(property "Reference" "FID2"
@@
 		(in_bom no)
 		(on_board yes)
-		(dnp no)
+		(dnp yes)
 		(fields_autoplaced yes)
 		(property "Reference" "FID5"
@@
 		(in_bom no)
 		(on_board yes)
-		(dnp no)
+		(dnp yes)
 		(fields_autoplaced yes)
 		(property "Reference" "FID1"

Commit message: First commit with 0.1mm traces and 02mm by 0.43mm vias to fit pcbway standard manufacturing + corrections of PR'S like uart RX of component to TX of mcu
Parts:
- removed APS6404L-SQH-SN1: PSRAM, footprint:APS6404L, symbol APS6404L-3SQR-SN:APS6404L-3SQR-SN
- removed C4: 0.22uF, Resistor_SMD:R_0603_1608Metric_Pad0.98x0.95mm_HandSolder, symbol Device:C
Connections:
- net Cam_RX: now also MIMXRT1062DVL6B1.C5 (GPIO_EMC_31); no longer MIMXRT1062DVL6B1.D5 (GPIO_EMC_32)
- net Cam_TX: now also MIMXRT1062DVL6B1.D5 (GPIO_EMC_32); no longer MIMXRT1062DVL6B1.C5 (GPIO_EMC_31)
- net Reserve_RX: now also MIMXRT1062DVL6B1.D13 (GPIO_B1_12); no longer MIMXRT1062DVL6B1.D14 (GPIO_B1_13)
- net Reserve_TX: now also MIMXRT1062DVL6B1.D14 (GPIO_B1_13); no longer MIMXRT1062DVL6B1.D13 (GPIO_B1_12)
- net Xbee_RX: now also MIMXRT1062DVL6B1.M11 (GPIO_AD_B0_02); no longer MIMXRT1062DVL6B1.G11 (GPIO_AD_B0_03)
- net Xbee_TX: now also MIMXRT1062DVL6B1.G11 (GPIO_AD_B0_03); no longer MIMXRT1062DVL6B1.M11 (GPIO_AD_B0_02)
- net BMO085_SCL renamed BNO085_SCL
- net BMO085_SDA renamed BNO085_SDA
- net EMC_24: no longer names the net of MIMXRT1062DVL6B1.D3 (GPIO_EMC_24)
- net EMC_25: no longer names the net of MIMXRT1062DVL6B1.D2 (GPIO_EMC_25)
- net EMC_26: no longer names the net of MIMXRT1062DVL6B1.B3 (GPIO_EMC_26)
- net EMC_27: no longer names the net of MIMXRT1062DVL6B1.A2 (GPIO_EMC_27)
- net EMC_28: no longer names the net of MIMXRT1062DVL6B1.D1 (GPIO_EMC_28)
- net EMC_29: no longer names the net of MIMXRT1062DVL6B1.E1 (GPIO_EMC_29)
- no-connect marks 87 -> 93
Other:
- sheet IMU BNO085 ports: added BNO085_SCL, BNO085_SDA; removed BMO085_SCL, BMO085_SDA
- note added: "RX 28"
- note added: "RX 34"
- note added: "Shortage, wait for PJRC to make BOOTLOADER compatible with possibly new flash"
- note added: "TX 29"
- note added: "TX 35"
- note removed: "28"
- note removed: "29"
- note removed: "34"
- note removed: "35"
- note removed: "Additional PSRAM (https://www.pjrc.com/store/psram.html)"
- note removed: "Check for 128mb storage"
