File: RocketFlightComputer/main/main.kicad_sch (KiCad schematic)
At the start: 66 parts, among them Y1 32.768kHz, Y5 XRCGB24M000F2P29R0

Commit message: Corrected a few subsystems
Connections:
- net BNO085_RST: now reaches MIMXRT1062DVL6B1.C3 (GPIO_EMC_36)
- no-connect marks 92 -> 91
Other:
- sheet IMU BNO085 ports: added BNO085_RST; removed none
- note added: "18"
- note added: "19"
- note added: "25"
- note added: "Permanent pull up high Pull down for rst"
Changed lines of the file:
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@@
 	)
 	(circle
+		(center 271.145 85.09)
+		(radius 0.635)
+		(stroke
+			(width 0)
+			(type default)
+		)
+		(fill
+			(type none)
+		)
+	)
+	(circle
 		(center 285.496 151.384)
 		(radius 0.635)
@@
 	)
 	(circle
+		(center 271.145 118.11)
+		(radius 0.635)
+		(stroke
+			(width 0)
+			(type default)
+		)
+		(fill
+			(type none)
+		)
+	)
+	(circle
 		(center 285.242 148.844)
 		(radius 0.635)
@@
 	)
 	(circle
+		(center 271.145 120.65)
+		(radius 0.635)
+		(stroke
+			(width 0)
+			(type default)
+		)
+		(fill
+			(type none)
+		)
+	)
+	(circle
 		(center 284.226 174.244)
 		(radius 0.635)
@@
 		)
 	)
+	(text "VERIFIED"
+		(exclude_from_sim no)
+		(at 422.148 129.286 0)
+		(effects
+			(font
+				(size 1 1)
+				(thickness 0.4)
+				(bold yes)
+			)
+			(justify left bottom)
+		)
+	)
 	(text "24"
 		(exclude_from_sim no)
@@
 		)
 	)
+	(text "VERIFIED"
+		(exclude_from_sim no)
+		(at 469.9 66.294 0)
+		(effects
+			(font
+				(size 1 1)
+				(thickness 0.4)
+				(bold yes)
+			)
+			(justify left bottom)
+		)
+	)
 	(text "23"
 		(exclude_from_sim no)
@@
 		)
 	)
+	(text "VERIFIED"
+		(exclude_from_sim no)
+		(at 469.138 95.758 0)
+		(effects
+			(font
+				(size 1 1)
+				(thickness 0.4)
+				(bold yes)
+			)
+			(justify left bottom)
+		)
+	)
 	(text "2.55ma to LED"
 		(exclude_from_sim no)
@@
 		)
 	)
+	(text "18"
+		(exclude_from_sim no)
+		(at 272.288 121.666 0)
+		(effects
+			(font
+				(size 1.27 1.27)
+			)
+			(justify left bottom)
+		)
+	)
 	(text "Not necessary \n(no external usb)"
 		(exclude_from_sim no)
@@
 		)
 	)
+	(text "VERIFIED"
+		(exclude_from_sim no)
+		(at 421.894 160.274 0)
+		(effects
+			(font
+				(size 1 1)
+				(thickness 0.4)
+				(bold yes)
+			)
+			(justify left bottom)
+		)
+	)
 	(text "Batt(17V to 3.3V) to 3.3V regulator (max 1.5A)"
 		(exclude_from_sim no)
@@
 		)
 	)
+	(text "VERIFIED"
+		(exclude_from_sim no)
+		(at 423.164 68.58 0)
+		(effects
+			(font
+				(size 1 1)
+				(thickness 0.4)
+				(bold yes)
+			)
+			(justify left bottom)
+		)
+	)
 	(text "41"
 		(exclude_from_sim no)
@@
 		)
 	)
+	(text "VERIFIED"
+		(exclude_from_sim no)
+		(at 466.852 130.302 0)
+		(effects
+			(font
+				(size 1 1)
+				(thickness 0.4)
+				(bold yes)
+			)
+			(justify left bottom)
+		)
+	)
 	(text "TX 29"
 		(exclude_from_sim no)
@@
 		)
 	)
+	(text "VERIFIED"
+		(exclude_from_sim no)
+		(at 13.97 214.884 0)
+		(effects
+			(font
+				(size 1 1)
+				(thickness 0.4)
+				(bold yes)
+			)
+			(justify left bottom)
+		)
+	)
 	(text "36"
 		(exclude_from_sim no)
@@
 		)
 	)
+	(text "VERIFIED"
+		(exclude_from_sim no)
+		(at 422.656 34.544 0)
+		(effects
+			(font
+				(size 1 1)
+				(thickness 0.4)
+				(bold yes)
+			)
+			(justify left bottom)
+		)
+	)
 	(text "40"
 		(exclude_from_sim no)
@@
 		)
 	)
+	(text "VERIFIED"
+		(exclude_from_sim no)
+		(at 423.672 96.774 0)
+		(effects
+			(font
+				(size 1 1)
+				(thickness 0.4)
+				(bold yes)
+			)
+			(justify left bottom)
+		)
+	)
 	(text "16"
 		(exclude_from_sim no)
@@
 		)
 	)
+	(text "Permanent pull up high\nPull down for rst"
+		(exclude_from_sim no)
+		(at 317.754 100.33 0)
+		(effects
+			(font
+				(size 0.7 0.7)
+			)
+			(justify left bottom)
+		)
+	)
 	(text "RX 34"
 		(exclude_from_sim no)
@@
 		)
 	)
+	(text "VERIFIED"
+		(exclude_from_sim no)
+		(at 468.884 35.814 0)
+		(effects
+			(font
+				(size 1 1)
+				(thickness 0.4)
+				(bold yes)
+			)
+			(justify left bottom)
+		)
+	)
 	(text "38"
 		(exclude_from_sim no)
@@
 		)
 	)
-	(text "21"
+	(text "25"
 		(exclude_from_sim no)
 		(at 272.415 165.1 0)
@@
 		)
 	)
+	(text "19"
+		(exclude_from_sim no)
+		(at 272.542 85.852 0)
+		(effects
+			(font
+				(size 1.27 1.27)
+			)
+			(justify left bottom)
+		)
+	)
 	(text "9"
 		(exclude_from_sim no)
@@
 	)
 	(no_connect
-		(at 303.53 100.33)
-	)
-	(no_connect
 		(at 303.53 54.61)
 	)
@@
 	(wire
 		(pts
+			(xy 392.43 106.68) (xy 406.4 106.68)
+		)
+		(stroke
+			(width 0)
+			(type default)
+		)
+	)
+	(wire
+		(pts
 			(xy 63.5 387.35) (xy 63.5 384.81)
 		)
@@
 	(wire
 		(pts
+			(xy 316.23 100.33) (xy 303.53 100.33)
+		)
+		(stroke
+			(width 0)
+			(type default)
+		)
+	)
+	(wire
+		(pts
 			(xy 499.11 212.09) (xy 483.87 212.09)
 		)
@@
 		)
 	)
+	(label "BNO085_RST"
+		(at 316.23 100.33 180)
+		(effects
+			(font
+				(size 1.27 1.27)
+			)
+			(justify right bottom)
+		)
+	)
 	(label "Reserve_TX"
 		(at 392.43 165.1 0)
@@
 		)
 	)
+	(label "BNO085_RST"
+		(at 392.43 106.68 0)
+		(effects
+			(font
+				(size 1.27 1.27)
+			)
+			(justify left bottom)
+		)
+	)
 	(label "PyroCH3_4"
 		(at 499.11 229.87 180)
@@
 			(effects
 				(font
+					(size 1.27 1.27)
+				)
+				(justify left)
+			)
+		)
+		(pin "BNO085_RST" bidirectional
+			(at 406.4 106.68 180)
+			(effects
+				(font

Commit message: Corrections of mistake, revision of schematic is done and BOM revised, revision of pcb layout to do
Parts:
- C17: value 0.22uF -> 10nF; LCSC C106216 -> C149619
- C7: value 10nF -> 10uF; LCSC C149619 -> C70225
- R1, R2: LCSC C1647 -> C22356467
- R4: value 1k -> 470; LCSC C21190 -> C23179
Connections:
- net GNDREF: now also C10.1, C9.2; no longer C10.2, MIMXRT1062DVL6B1.P9 (RTC_XTALO), Y1.1, Y5.3 (XTAL_2), Y5.4 (NC_2)
- net N11: now also Y5.3 (XTAL_2); no longer Y5.2 (NC_1)
- net 3.3v_led: no longer names the net of D1.1 (K), R4.2
- new net: C10.2, MIMXRT1062DVL6B1.P9 (RTC_XTALO), Y1.1
- no-connect marks 91 -> 93
Other:
- note added: "Fixed 3.3v output version"
- note added: "Not necessary (output enable for peripheral usb)"
- note added: "Sense when USB connected with 5v"
- note removed: "Sense when USB connected"
- moved on the sheet: C1, C2, C3, D1, L1, R3, R4

Commit message: Because i am lazy i would call this the V1 of the avionics
Parts:
- Y5: footprint XRCGB -> footprint:XRCGB
Changed lines of the file:
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@@
 			)
 		)
-		(property "Footprint" "XRCGB"
+		(property "Footprint" "footprint:XRCGB"
 			(at 369.24 298.45 0)
 			(hide yes)

Commit message: Was missing pull ups on adxl375
Connections:
- net GNDREF: now also MIMXRT1062DVL6B1.K9 (NGND_KEL0)
- no-connect marks 93 -> 92
Changed lines of the file:
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@@
 	)
 	(no_connect
-		(at 250.19 115.57)
-	)
-	(no_connect
 		(at 250.19 46.99)
 	)
@@
 					(unit 1)
 				)
+			)
+		)
+	)
+	(symbol
+		(lib_id "power:GNDREF")
+		(at 250.19 115.57 270)
+		(mirror x)
+		(unit 1)
+		(body_style 1)
+		(exclude_from_sim no)
+		(in_bom yes)
+		(on_board yes)
+		(in_pos_files yes)
+		(dnp no)
+		(fields_autoplaced yes)
+		(property "Reference" "#PWR087"
+			(at 243.84 115.57 0)
+			(hide yes)
+			(show_name no)
+			(do_not_autoplace no)
+			(effects
+				(font
+					(size 1.27 1.27)
+				)
+			)
+		)
+		(property "Value" "GNDREF"
+			(at 246.38 116.205 90)
+			(hide yes)
+			(show_name no)
+			(do_not_autoplace no)
+			(effects
+				(font
+					(size 1.27 1.27)
+				)
+				(justify right)
+			)
+		)
+		(property "Footprint" ""
+			(at 250.19 115.57 0)
+			(hide yes)
+			(show_name no)
+			(do_not_autoplace no)
+			(effects
+				(font
+					(size 1.27 1.27)
+				)
+			)
+		)
+		(property "Datasheet" ""
+			(at 250.19 115.57 0)
+			(hide yes)
+			(show_name no)
+			(do_not_autoplace no)
+			(effects
+				(font
+					(size 1.27 1.27)
+				)
+			)
+		)
+		(property "Description" ""
+			(at 250.19 115.57 0)
+			(hide yes)
+			(show_name no)
+			(do_not_autoplace no)
+			(effects
+				(font
+					(size 1.27 1.27)
+				)
+			)
+		)
+		(pin "1"
+		)
+		(instances
+			(project "main"
+				(path "/27195d1d-92b2-40df-ada5-3b20841577e7"
+					(reference "#PWR087")
+					(unit 1)
+				)

Commit message: REVA board?
Parts:
- MKL02Z32VFG1: now fitted
Changed lines of the file:
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@@
 		(on_board yes)
 		(in_pos_files yes)
-		(dnp yes)
+		(dnp no)
 		(property "Reference" "MKL02Z32VFG1"
 			(at 187.96 322.58 0)
