File: RocketFlightComputer/main/_autosave-HighCurrentComponents.kicad_sch.kicad_sch (KiCad schematic)
At the start: 23 parts, among them J1 BATT, Q2 SI2302, Q3 SI2302, Q4 SI2302

Commit message: Layout changes to incorporate power capacitors for the servos
Parts:
- C41: footprint Capacitor_SMD:CP_Elec_5x5.8 -> Capacitor_SMD:C_1210_3225Metric_Pad1.33x2.70mm_HandSolder
Changed lines of the file:
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@@
 			)
 		)
-		(property "Footprint" "Capacitor_SMD:CP_Elec_5x5.8"
+		(property "Footprint" "Capacitor_SMD:C_1210_3225Metric_Pad1.33x2.70mm_HandSolder"
 			(at 239.7252 140.97 0)
 			(effects
