File: RocketFlightComputer/main/ADXL375.kicad_sch (KiCad schematic)
At the start: 4 parts

Commit message: Corrected a few subsystems
Other:
- note added: "Ceramic capacitor"
- note added: "Tantalum capacitor"
Changed lines of the file:
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@@
 	(generator_version "10.0")
 	(paper "User" 150.012 150.012)
+	(text "Tantalum capacitor"
+		(exclude_from_sim no)
+		(at 36.576 46.99 0)
+		(effects
+			(font
+				(size 0.7 0.7)
+			)
+			(justify left bottom)
+		)
+	)
 	(text "Max current: 145 uA\n"
 		(exclude_from_sim no)
@@
 			)
 			(justify left bottom)
+		)
+	)
+	(text "Ceramic capacitor"
+		(exclude_from_sim no)
+		(at 36.83 58.42 0)
+		(effects
+			(font
+				(size 0.7 0.7)
+			)
+			(justify left bottom)
