File: RocketFlightComputer/main/telemetry.kicad_sch (KiCad schematic)
At the start: 1 part

Commit message: REVA board?
Parts:
- renumbered S4B-PH-K-S_LF__SN_1 to JST-GH-1
Changed lines of the file:
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@@
 		(in_pos_files yes)
 		(dnp no)
-		(property "Reference" "S4B-PH-K-S_LF__SN_1"
+		(property "Reference" "JST-GH-1"
 			(at 80.264 53.086 0)
 			(hide yes)
@@
 			(project "main"
 				(path "/27195d1d-92b2-40df-ada5-3b20841577e7/e28c6e59-b6f8-4de5-b42d-020f37d4635d"
-					(reference "S4B-PH-K-S_LF__SN_1")
+					(reference "JST-GH-1")
 					(unit 1)
 				)
