File: PCB/main/main.kicad_pcb (KiCad board)
At the start: 4 copper layers, 53.7 x 53.7 mm, 131 parts, among them Q1 DMG3406L, Q2 DMG3406L, Q3 DMG3406L, Y1 32.768kHz, Y3 32.768kHz, Y4 32.768kHz, Y5 XRCGB24M000F2P29R0

Commit message: Servos, camera and telemetry connection (telemetry needs work, only one way comms for now)
Parts:
- added ?: , , F.Cu at (120.0, 43.1)
- added REF**: MountingHole_2.5mm, MountingHole:MountingHole_2.5mm, F.Cu at (92.8, 63.2)
Routing:
- net /BMP390_SDA1: track 65.1 -> 67.0 mm
